Commit message: Update joint origin rotation for camera model

File: depthai_descriptions/urdf/include/base_macro.urdf.xacro (robot description, xacro)
@@ -58,5 +58,5 @@
 			<parent link="${base_frame}" />
 			<child link="${camera_name}_model_origin" />
-			<origin xyz="0 0 0" rpy="1.5708 0 1.5708" />
+			<origin xyz="0 0 0" rpy="0 0 ${M_PI}" />
 		</joint>
 		<!-- IMU -->
