Commit message: Update joint origins for camera configuration

File: depthai_descriptions/urdf/include/depthai_macro.urdf.xacro (robot description, xacro)
@@ -45,5 +45,5 @@
 			<link name="${camera_name}_${rgb_name}_${optical_frame_suffix}" />
 			<joint name="${camera_name}_rgb_camera_optical_joint" type="fixed">
-				<origin xyz="0 0 0" rpy="-${M_PI/2} 0.0 -${M_PI/2}" />
+				<origin xyz="0 0 0" rpy="0 0.0 0" />
 				<parent link="${camera_name}_${rgb_name}_${frame_suffix}" />
 				<child link="${camera_name}_${rgb_name}_${optical_frame_suffix}" />
@@ -85,9 +85,9 @@
 				<parent link="${base_frame}" />
 				<child link="${camera_name}_${left_name}_${frame_suffix}" />
-				<origin xyz="0 0.1 0" rpy="0 0 0" />
+				<origin xyz="-0.1 0 0" rpy="0 0 0" />
 			</joint>
 			<link name="${camera_name}_${left_name}_${optical_frame_suffix}" />
 			<joint name="${camera_name}_left_camera_optical_joint" type="fixed">
-				<origin xyz="0 0 0" rpy="-${M_PI/2} 0.0 -${M_PI/2}" />
+				<origin xyz="0 0 0" rpy="0 0.0 0" />
 				<parent link="${camera_name}_${left_name}_${frame_suffix}" />
 				<child link="${camera_name}_${left_name}_${optical_frame_suffix}" />
@@ -98,9 +98,9 @@
 				<parent link="${base_frame}" />
 				<child link="${camera_name}_${right_name}_${frame_suffix}" />
-				<origin xyz="0 -0.05 0" rpy="0 0 0" />
+				<origin xyz="0.05 0 0" rpy="0 0 0" />
 			</joint>
 			<link name="${camera_name}_${right_name}_${optical_frame_suffix}" />
 			<joint name="${camera_name}_right_camera_optical_joint" type="fixed">
-				<origin xyz="0 0 0" rpy="-${M_PI/2} 0.0 -${M_PI/2}" />
+				<origin xyz="0 0 0" rpy="0 0.0 0" />
 				<parent link="${camera_name}_${right_name}_${frame_suffix}" />
 				<child link="${camera_name}_${right_name}_${optical_frame_suffix}" />
